File: electronics/butterfly-chonky/butterfly-chonky.kicad_sch (KiCad schematic)
At the start: 21 parts, among them J1 Conn_01x04_Pin, J2 Conn_01x03_Pin, J3 Conn_01x03_Pin, J4 Conn_01x03_Pin, Q1 2N2222, SW1 SW_Push, SW2 SW_Push, SW3 Switch_Header, U1 MPU6050_Module

Commit message: Zweeeop, ZweeeeeeOP, zwoop zwuup
Parts:
- removed J1: Conn_01x04_Pin, Connector_PinHeader_2.54mm:PinHeader_1x04_P2.54mm_Horizontal, symbol Connector:Conn_01x04_Pin
- added J1: Conn_02x06_Odd_Even, Connector_PinHeader_2.54mm:PinHeader_2x06_P2.54mm_Vertical_SMD, symbol Connector_Generic:Conn_02x06_Odd_Even
- added J5: Conn_01x04_Socket, Connector_PinHeader_2.54mm:PinHeader_1x04_P2.54mm_Vertical, symbol Connector:Conn_01x04_Socket
- added J6: Conn_01x03_Pin, Connector_PinHeader_2.54mm:PinHeader_1x03_P2.54mm_Vertical, symbol Connector:Conn_01x03_Pin
- added JP1, JP2: SolderJumper_2_Bridged, Jumper:SolderJumper-2_P1.3mm_Bridged_RoundedPad1.0x1.5mm, symbol Jumper:SolderJumper_2_Bridged
- added R7: A9050, OptoDevice:R_LDR_5.0x4.1mm_P3mm_Vertical, symbol Sensor_Optical:A9050
- added R8, R9: 10k, Resistor_THT:R_Axial_DIN0204_L3.6mm_D1.6mm_P7.62mm_Horizontal, symbol Device:R
- added U2: DHT11_Module, !RobotButterfly:DHT11_Module, symbol !RobotButterfly:DHT11_Module
- added U3: Mic_Module, !RobotButterfly:Mic_Module, symbol !RobotButterfly:Mic_Module
- BZ1: Digikey (none) -> 445-2525-1-ND; Digikey2 (none) -> 445-5242-1-ND
- D1, D2: Digikey (none) -> 365-1183-ND
- M1: footprint !RobotButterfly:Boostlet_v1.2 -> !RobotButterfly:Boostlet_v1.3; symbol !RobotButterfly:Boostlet_v1.2 -> !RobotButterfly:Boostlet_v1.3
- M2: footprint !RobotButterfly:Keystone-ESP_v1.1 -> !RobotButterfly:Keystone-ESP_v1.2; symbol !RobotButterfly:Keystone-ESP_v1.1 -> !RobotButterfly:Keystone-ESP_v1.2
- PS1: footprint !RobotButterfly:2xAA_Battery_Module -> !RobotButterfly:Batt_Header
- Q1: Digikey 641-1942-1-ND -> PN2222AFS-ND; Digikey2 (none) -> 1514-PN2222APBFREE-ND
- R1: Digikey RMCF1206FT2K00CT-ND -> CF14JT2K00CT-ND
- R2, R4: Digikey (none) -> CF14JT10K0CT-ND
- R3: Digikey 13-RC1206FR-10330RLCT-ND -> CF14JT330RCT-ND
- R5, R6: Digikey (none) -> CF14JT330RCT-ND
- SW2: renamed from SW1; Digikey (none) -> EG5994-ND; Digikey2 (none) -> 486-3460-ND
- SW3: renamed from SW2; Digikey (none) -> EG5994-ND; Digikey2 (none) -> 486-3460-ND
- renumbered SW3 to SW1
Connections:
- net 5V: now also J1.11 (Pin_11)
- net BUTTON_3: now also J1.9 (Pin_9)
- net GND: now also J1.1 (Pin_1), J1.12 (Pin_12), J5.1 (Pin_1), J6.1 (Pin_1), R9.1, U2.4 (Gnd), U3.2 (Gnd)
- net LDR: now also R7.2, R9.2
- net MIC: now also U3.1 (Sig)
- net PROXIMITY_L: now also J1.5 (Pin_5), JP1.1 (A)
- net PROXIMITY_R: now also J1.7 (Pin_7), JP2.2 (B)
- net SCL: now also J1.2 (Pin_2)
- net SDA: now also J1.4 (Pin_4)
- net SERVO_L: now also M2.5 (IO19); no longer M2.2 (IO23)
- net SERVO_R: now also M2.2 (IO23); no longer M2.5 (IO19)
- net SERVO_X: now also J1.6 (Pin_6)
- net UART2_RX: now also J1.10 (Pin_10)
- net UART2_TX: now also J1.8 (Pin_8)
- net ULTRASONIC_IN: now also J5.2 (Pin_2)
- net ULTRASONIC_OUT: now also J5.3 (Pin_3)
- net VCC: now also J1.3 (Pin_3), J5.4 (Pin_4), J6.2 (Pin_2), R7.1, R8.2, U2.1 (Vcc), U3.3 (Vcc)
- new net: J6.3 (Pin_3), JP1.2 (B)
- new net: JP2.1 (A), R8.1, U2.2 (Data)
Other:
- note added: "Aux Header"
- note added: "LDR"
- note added: "Robot Butterfly (C) Copyright Erin RobotZwrrl, Robot Missions Inc. 04-11-24 v1.1 RobotZwrrl.xyz RobotMissions.org This hardware is released under: CERN Open Hardware License Version 2.0 - Permissive (CERN-OHL-P) Disclaimer: Distributed as is. No warranty is given. Not responsible or liable for any damage or harm that result from this product."
- note added: "TODO: Organise this"
- note added: "gnd 32 33 22 21 18 17 16 15 vcc 5v gnd"
- note removed: "Butterfly-Chonky (C) Copyright Erin RobotZwrrl, Robot Missions Inc. 03-16-24 v1.0 RobotZwrrl.xyz RobotMissions.org This hardware is released under: CERN Open Hardware License Version 2.0 - Permissive (CERN-OHL-P) Disclaimer: Distributed as is. No warranty is given. Not responsible or liable for any damage or harm that result from this product."
- moved on the sheet: BZ1, D1, D2, Q1, R1, R2, R3, R4, R5, R6, SW2, SW3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
