File: electronics/butterfly-chonky/archive/butterfly-chonky.kicad_sch (KiCad schematic)
At the start: 30 parts, among them J1 Conn_02x06_Odd_Even, J2 Conn_01x03_Pin, J3 Conn_01x03_Pin, J4 Conn_01x03_Pin, J5 Conn_01x04_Socket, J6 Conn_01x03_Pin, Q1 2N2222, SW1 Switch_Header, SW2 SW_Push, SW3 SW_Push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

Commit message: Organised schematic
Other:
- note added: "LDR"
- note added: "Robot Butterfly (C) Copyright Erin RobotZwrrl, Robot Missions Inc. 04-11-24 v1.1 RobotZwrrl.xyz RobotMissions.org This hardware is released under: CERN Open Hardware License Version 2.0 - Permissive (CERN-OHL-P) Disclaimer: Distributed as is. No warranty is given. Not responsible or liable for any damage or harm that result from this product."
- note added: "TODO: Organise this"
- note added: "gnd 32 33 22 21 18 17 16 15 vcc 5v gnd"
- note removed: "Disclaimer: Distributed as is. No warranty is given. Not responsible or liable for any damage or harm that result from this product."
- note removed: "Robot Butterfly (C) Copyright Erin RobotZwrrl, Robot Missions Inc. 04-11-24 v1.1 RobotZwrrl.xyz RobotMissions.org"
- note removed: "This hardware is released under: CERN Open Hardware License Version 2.0 - Permissive (CERN-OHL-P)"
- moved on the sheet: BZ1, D1, D2, J1, J2, J3, J4, J5, J6, JP1, JP2, M1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
